File: Hardware/MCU.kicad_sch (KiCad schematic)
At the start: 0 parts

Commit message: complete sch
Parts:
- added C102, C104, C105, C106, C107, C108: 100nF, persional_library:C0603, symbol persional_library:C0603
- added R78, R79, R80: 10kΩ, persional_library:R0603, symbol persional_library:R0603
- added SW1: ~, persional_library:SW-SMD_4P-L4.2-W3.2-P2.15-LS4.6-1, symbol persional_library:Switch_PushButton_TS3425BA
- added U17: ~, persional_library:LQFP-48_L7.0-W7.0-P0.50-LS9.0-BL, symbol persional_library:STM32F103CBT6
- added U18: ~, persional_library:CONN-SMD_4P-P1.25_XUNPU_WAFER-GH1.25-4PWB, symbol persional_library:Connect_GH1.25_4P_Horizontal
- added X2: 8MHz, persional_library:OSC-SMD_3P-L3.2-W1.3-P1.20-L, symbol persional_library:XTAL_8MHz_NP
Connections:
- new net: R79.2, U17.20 (PB2BOOT1)
- new net: R78.1, U17.44 (BOOT0)
- new net +3.3V: C102.2, C104.2, C105.2, C106.2, C107.2, R80.2, U17.1 (VBAT), U17.24 (VDD_1), U17.36 (VDD_2), U17.48 (VDD_3), U17.9 (VDD_A), U18.4
- new net Connect_RX: U17.31 (PA10USART1_RXTIM1_CH3)
- new net Connect_TX: U17.30 (PA9USART1_TXTIM1_CH2)
- new net GND: C102.1, C104.1, C105.1, C106.1, C107.1, C108.2, R78.2, R79.1, SW1.4, U17.23 (VSS_1), U17.35 (VSS_2), U17.47 (VSS_3), U17.8 (VSS_A), U18.1, U18.5, U18.6, X2.2 (GND)
- new net GPIO_1: U17.21 (PB10I2C2_SCLUSART3_TX)
- new net GPIO_2: U17.22 (PB11I2C2_SDAUSART3_RX-)
- new net HDMI_KEY: U17.25 (PB12SPI2_NSSI2C2_SMBAUSART3_CKTIM1_BKIN)
- new net HMDI_EN: U17.41 (PB5I2C1_SMBA)
- new net HMDI_SEL1: U17.40 (PB4NJTRST)
- new net HMDI_SEL2: U17.39 (PB3JTDO)
- new net HUB_KEY1: U17.29 (PA8USART1_CKTIM1_CH1MCO)
- new net HUB_KEY2: U17.28 (PB15SPI2_MOSITIM1_CH3N)
- new net HUB_KEY3: U17.27 (PB14SPI2_MISOUSART3_RTSTIM1_CH2N)
- new net HUB_KEY4: U17.26 (PB13SPI2_SCKUSART3_CTSTIM1_CH1N)
- new net HUB_SEL0: U17.33 (PA12USART1_RTSCAN_TXTIM1_ETRUSBDP)
- new net HUB_SEL1: U17.32 (PA11USART1_CTSCAN_RXTIM1_CH4USBDM)
- new net I2C_SCL: U17.42 (PB6I2C1_SCLTIM4_CH1)
- new net I2C_SDA: U17.43 (PB7I2C1_SDATIM4_CH2)
- new net OSC_IN: U17.5 (PD0-OSC_IN), X2.1 (OSC1)
- new net OSC_OUT: U17.6 (PD1-OSC_OUT), X2.3 (OSC2)
- new net RST: C108.1, R80.1, SW1.2, U17.7 (NRST)
- new net SWCLK: U17.37 (PA14JTCKSWCLK), U18.3
- new net SWDIO: U17.34 (PA13JTMSSWDIO), U18.2
- new net USART2_RX: U17.13 (PA3USART2_RXADC12_IN3TIM2_CH4)
- new net USART2_TX: U17.12 (PA2USART2_TXADC12_IN2TIM2_CH3)
- no-connect marks 0 -> 15

Commit message: 修改了一些小错误,并补充部分外设
Parts:
- added C110, C111, C112, C113, C114, C115: 100nF, persional_library:C0603, symbol persional_library:C0603
- added CN1: ~, persional_library:CONN-TH_3P-P1.25_GH1.25, symbol persional_library:Connect_GH1.25_3P_Horizontal
- added H1, H2: ~, persional_library:HDR-TH_4P-P2.54-V-M, symbol persional_library:Connect_XH2.54_1x4P
- added R92, R93, R94, R95, R96, R97: 10kΩ, persional_library:R0603, symbol persional_library:R0603
- added SW2, SW3, SW4, SW5, SW6, SW7: ~, persional_library:SW-SMD_4P-L4.2-W3.2-P2.15-LS4.6-1, symbol persional_library:Switch_PushButton_TS3425BA
Connections:
- net +3.3V: now also H1.1, H2.3, R92.2, R93.2, R94.2, R95.2, R96.2, R97.2
- net Connect_RX: now also CN1.1
- net Connect_TX: now also CN1.2
- net GND: now also C110.2, C111.2, C112.2, C113.2, C114.2, C115.2, CN1.3, CN1.4, CN1.5, H1.2, H2.4, SW2.4, SW3.4, SW4.4, SW5.4, SW6.4, SW7.4
- net HDMI_KEY: now also C113.1, R95.1, SW5.2
- net HMDI_EN: now also U17.19 (PB1ADC12_IN9TIM3_CH4), C115.1, R97.1, SW7.2
- net HUB_KEY1: now also C110.1, R92.1, SW2.2
- net HUB_KEY2: now also C112.1, R94.1, SW4.2
- net HUB_KEY3: now also C114.1, R96.1, SW6.2
- net HUB_KEY4: now also C111.1, R93.1, SW3.2
- net I2C_SCL: now also H2.2
- net I2C_SDA: now also H2.1
- net USART2_RX: now also H1.4
- net USART2_TX: now also H1.3
- no-connect marks 15 -> 26
