File: Hardware/ChinoHub.kicad_pcb (KiCad board)
At the start: 2 copper layers, 8.2 x 0.8 mm, 236 parts, among them X1 25MHz

Commit message: 修改了一些小错误,并补充部分外设
Parts:
- added C103: 1uF, persional_library:C0603, F.Cu at (168.6, 32.5)
- added C104: 100nF, persional_library:C0603, F.Cu at (134.3, 27.6)
- added C105: 100nF, persional_library:C0603, F.Cu at (134.3, 30.2)
- added C106: 100nF, persional_library:C0603, F.Cu at (134.3, 32.9)
- added C107: 100nF, persional_library:C0603, F.Cu at (134.3, 35.6)
- added C108: 100nF, persional_library:C0603, F.Cu at (134.3, 38.3)
- added C109: 100nF, persional_library:C0603, F.Cu at (131.7, 64.0)
- added C110: 100nF, persional_library:C0603, F.Cu at (134.3, 40.9)
- added C111: 100nF, persional_library:C0603, F.Cu at (138.3, 27.6)
- added C112: 100nF, persional_library:C0603, F.Cu at (138.3, 30.2)
- added C113: 100nF, persional_library:C0603, F.Cu at (138.3, 32.9)
- added C114: 100nF, persional_library:C0603, F.Cu at (138.3, 35.6)
- added C115: 100nF, persional_library:C0603, F.Cu at (138.3, 38.3)
- added CN1: ~, persional_library:CONN-TH_3P-P1.25_GH1.25, F.Cu at (148.3, 29.2)
- added D6: ~, persional_library:SMB_L4.6-W3.6-LS5.3-RD, F.Cu at (166.2, 41.3)
- added D7: ~, persional_library:SOD-323F_L1.7-W1.3-LS2.5-R-RD, F.Cu at (162.7, 49.6)
- added D8: ~, persional_library:SOD-323F_L1.7-W1.3-LS2.5-R-RD, F.Cu at (131.8, 61.4)
- added D9: ~, persional_library:SOD-323F_L1.7-W1.3-LS2.5-R-RD, F.Cu at (162.7, 52.2)
- added F1: ~, persional_library:F1206, F.Cu at (159.5, 27.9)
- added F2: ~, persional_library:F1206, F.Cu at (159.5, 31.2)
- added F3: ~, persional_library:F1206, F.Cu at (159.5, 34.6)
- added F4: ~, persional_library:F1206, F.Cu at (159.5, 37.9)
- added F5: ~, persional_library:F1206, F.Cu at (159.5, 41.2)
- added F6: ~, persional_library:F1206, F.Cu at (159.5, 44.6)
- added H1: ~, persional_library:HDR-TH_4P-P2.54-V-M, F.Cu at (138.0, 44.2)
- added H2: ~, persional_library:HDR-TH_4P-P2.54-V-M, F.Cu at (138.0, 48.0)
- added Q16: ~, persional_library:SOT-23-3_L2.9-W1.3-P1.90-LS2.4-BR, F.Cu at (164.5, 28.3)
- added Q17: ~, persional_library:SOT-23-3_L2.9-W1.3-P0.95-LS2.4-BR-1, F.Cu at (164.5, 32.5)
- added Q18: ~, persional_library:SOT-23-3_L2.9-W1.3-P1.90-LS2.4-BR, F.Cu at (164.5, 36.7)
- added R82: 10K, persional_library:R0603, F.Cu at (168.6, 27.5)
- added R83: 47K, persional_library:R0603, F.Cu at (168.6, 29.9)
- added R84: 2.2kΩ, persional_library:R0603, F.Cu at (158.6, 49.5)
- added R85: 2.2kΩ, persional_library:R0603, F.Cu at (127.7, 61.3)
- added R86: 2.2kΩ, persional_library:R0603, F.Cu at (127.7, 63.7)
- added R87: 2.2kΩ, persional_library:R0603, F.Cu at (158.6, 52.0)
- added R88: 2.2kΩ, persional_library:R0603, F.Cu at (158.6, 54.4)
- added R89: 100kΩ, persional_library:R0603, F.Cu at (127.7, 66.2)
- added R90: 10kΩ, persional_library:R0603, F.Cu at (158.6, 56.9)
- added R91: 10kΩ, persional_library:R0603, F.Cu at (158.6, 59.4)
- added R92: 10kΩ, persional_library:R0603, F.Cu at (142.3, 27.5)
- added R93: 10kΩ, persional_library:R0603, F.Cu at (142.3, 29.9)
- added R94: 10kΩ, persional_library:R0603, F.Cu at (142.3, 32.4)
- added R95: 10kΩ, persional_library:R0603, F.Cu at (142.3, 34.9)
- added R96: 10kΩ, persional_library:R0603, F.Cu at (142.3, 37.4)
- added R97: 10kΩ, persional_library:R0603, F.Cu at (142.3, 39.8)
- added SW1: ~, persional_library:SW-SMD_4P-L4.2-W3.2-P2.15-LS4.6-1, F.Cu at (129.0, 28.5)
- added SW2: ~, persional_library:SW-SMD_4P-L4.2-W3.2-P2.15-LS4.6-1, F.Cu at (129.0, 33.0)
- added SW3: ~, persional_library:SW-SMD_4P-L4.2-W3.2-P2.15-LS4.6-1, F.Cu at (129.0, 37.6)
- added SW4: ~, persional_library:SW-SMD_4P-L4.2-W3.2-P2.15-LS4.6-1, F.Cu at (129.0, 42.1)
- added SW5: ~, persional_library:SW-SMD_4P-L4.2-W3.2-P2.15-LS4.6-1, F.Cu at (129.0, 46.7)
- added SW6: ~, persional_library:SW-SMD_4P-L4.2-W3.2-P2.15-LS4.6-1, F.Cu at (129.0, 51.2)
- added SW7: ~, persional_library:SW-SMD_4P-L4.2-W3.2-P2.15-LS4.6-1, F.Cu at (129.0, 55.8)
- added U17: ~, persional_library:LQFP-48_L7.0-W7.0-P0.50-LS9.0-BL, F.Cu at (149.2, 47.8)
- added U18: ~, persional_library:CONN-SMD_4P-P1.25_XUNPU_WAFER-GH1.25-4PWB, F.Cu at (137.0, 52.8)
- added X2: 8MHz, persional_library:OSC-SMD_3P-L3.2-W1.3-P1.20-L, F.Cu at (147.1, 34.3)
- C100, C97: value 1uF -> 10uF
- C101, C95: value 1uF -> 100nF
- C102: value 10uF -> 100nF
- R74: value 10kΩ -> 150K
- R75: value 100kΩ -> 150K
- R76: value 1MΩ -> 680K
- R77: value 220kΩ -> 100K
- R78, R80: value 100kΩ -> 10kΩ
- R81: value 150kΩ -> 2.2kΩ
- U15: footprint persional_library:SOT-23-5_L3.0-W1.7-P0.95-LS2.8-BR -> persional_library:TSOT-23-8_L2.9-W1.6-P0.65-LS2.8-BL
- U16: footprint persional_library:SOT-23-5_L3.0-W1.7-P0.95-LS2.8-BR -> persional_library:SOT-223-4_L6.5-W3.5-P2.30-LS7.0-BR
Connections:
- net /USB_HUB/SEL_0 renamed /MCU/HUB_SEL0
- net /USB_HUB/SEL_1 renamed /MCU/HUB_SEL1
- C100 pad 2: +5V -> +3.3V
- C101 pad 2: +1V0 -> +3.3V
- C102 pad 2: +1V0 -> +3.3V
- C17 pad 2: /TypeC3.0Handle/TypeC_1_5V -> /Power/TypeC_1_5V
- C18 pad 2: /TypeC3.0Handle/TypeC_1_5V -> /Power/TypeC_1_5V
- C19 pad 2: /TypeC3.0Handle/TypeC_2_5V -> /Power/TypeC_2_5V
- C20 pad 2: /TypeC3.0Handle/TypeC_2_5V -> /Power/TypeC_2_5V
- C21 pad 2: /TypeC3.0Handle/TypeC_3_5V -> /Power/TypeC_3_5V
- C22 pad 2: /TypeC3.0Handle/TypeC_3_5V -> /Power/TypeC_3_5V
- C23 pad 2: /TypeC3.0Handle/TypeC_4_5V -> /Power/TypeC_4_5V
- C24 pad 2: /TypeC3.0Handle/TypeC_4_5V -> /Power/TypeC_4_5V
- C82 pad 1: /OUT_HUB/HUB_5V -> +5V
- C83 pad 1: /OUT_HUB/HUB_5V -> +5V
- C84 pad 1: /OUT_HUB/HUB_5V -> +5V
- C85 pad 1: /OUT_HUB/HUB_5V -> +5V
- C86 pad 1: /OUT_HUB/HUB_5V -> +5V
- C87 pad 1: /OUT_HUB/HUB_5V -> +5V
- C88 pad 1: /OUT_HUB/HUB_5V -> +5V
- C89 pad 1: /OUT_HUB/HUB_5V -> +5V
- C90 pad 2: /Power/TypeC_1_5V -> Net-(Q1-D)
- C91 pad 2: /Power/TypeC_2_5V -> Net-(Q4-E)
- C92 pad 2: /Power/TypeC_3_5V -> Net-(Q7-E)
- C93 pad 2: /Power/TypeC_4_5V -> Net-(Q10-E)
- C94 pad 2: /Power/HDMI_VBUS -> Net-(Q13-E)
- C98 pad 2: +3V3 -> +1V0
- D1 pad 1: /Power/TypeC_1_5V -> Net-(Q1-D)
- D2 pad 1: /Power/TypeC_2_5V -> Net-(Q4-E)
- D3 pad 1: /Power/TypeC_3_5V -> Net-(Q7-E)
- D4 pad 1: /Power/TypeC_4_5V -> Net-(Q10-E)
- D5 pad 1: /Power/HDMI_VBUS -> Net-(Q13-E)
- L1 pad 1: Net-(U15-LX) -> Net-(U15-SW1)
- L2 pad 1: Net-(U16-LX) -> Net-(U15-SW2)
- Q1 pad 3: /Power/TypeC_1_5V -> Net-(Q1-D)
- Q10 pad 2: /Power/TypeC_4_5V -> Net-(Q10-E)
- Q11 pad 3: /Power/TypeC_4_5V -> Net-(Q10-E)
- Q13 pad 2: /Power/HDMI_VBUS -> Net-(Q13-E)
- Q14 pad 3: /Power/HDMI_VBUS -> Net-(Q13-E)
- Q2 pad 2: /Power/TypeC_1_5V -> Net-(Q1-D)
- Q4 pad 2: /Power/TypeC_2_5V -> Net-(Q4-E)
- Q5 pad 3: /Power/TypeC_2_5V -> Net-(Q4-E)
- Q7 pad 2: /Power/TypeC_3_5V -> Net-(Q7-E)
- Q8 pad 3: /Power/TypeC_3_5V -> Net-(Q7-E)
- R10 pad 2: /TypeC3.0Handle/TypeC_2_5V -> /Power/TypeC_2_5V
- R12 pad 2: /TypeC3.0Handle/TypeC_2_5V -> /Power/TypeC_2_5V
- R14 pad 2: /TypeC3.0Handle/TypeC_3_5V -> /Power/TypeC_3_5V
- R15 pad 2: /TypeC3.0Handle/TypeC_3_5V -> /Power/TypeC_3_5V
- R17 pad 2: /TypeC3.0Handle/TypeC_3_5V -> /Power/TypeC_3_5V
- R19 pad 2: /TypeC3.0Handle/TypeC_4_5V -> /Power/TypeC_4_5V
- R20 pad 2: /TypeC3.0Handle/TypeC_4_5V -> /Power/TypeC_4_5V
- R22 pad 2: /TypeC3.0Handle/TypeC_4_5V -> /Power/TypeC_4_5V
- R4 pad 2: /TypeC3.0Handle/TypeC_1_5V -> /Power/TypeC_1_5V
- R43 pad 2: /TypeC2HDMI/HDMI_5V -> +5V
- R5 pad 2: /TypeC3.0Handle/TypeC_1_5V -> /Power/TypeC_1_5V
- R6 pad 2: /TypeC3.0Handle/TypeC_1_5V -> /Power/TypeC_1_5V
- R74 pad 1: Net-(U15-EN) -> Net-(U15-FB2)
- R74 pad 2: +5V -> GND
- R75 pad 1: GND -> Net-(U15-FB1)
- R75 pad 2: Net-(U15-EN) -> GND
- R76 pad 1: Net-(U15-FB/Vout) -> Net-(U15-FB1)
- R77 pad 1: GND -> Net-(U15-FB2)
- R77 pad 2: Net-(U15-FB/Vout) -> +1V0
- R78 pad 1: GND -> Net-(U17-BOOT0)
- R78 pad 2: Net-(U16-EN) -> GND
- R79 pad 1: Net-(U16-EN) -> GND
- R79 pad 2: +5V -> Net-(U17-PB2BOOT1)
- R80 pad 1: Net-(U16-FB/Vout) -> /MCU/RST
- R80 pad 2: +1V0 -> +3.3V
- R81 pad 1: GND -> Net-(D7-Pad1)
- R81 pad 2: Net-(U16-FB/Vout) -> /HDMI_OUT/HDMI_SDA
- R9 pad 2: /TypeC3.0Handle/TypeC_2_5V -> /Power/TypeC_2_5V
- U10 pad 1: /OUT_HUB/HUB_5V -> +5V
- U11 pad 1: /OUT_HUB/HUB_5V -> +5V
- U12 pad 1: /OUT_HUB/HUB_5V -> +5V
- U13 pad 1: /OUT_HUB/HUB_5V -> +5V
- U14 pad 1: unconnected-(U14-VCC-Pad1) -> +3V3
- U14 pad 10: unconnected-(U14-D2+-Pad10) -> /HDMI_OUT/HDMI0_D1_N
- U14 pad 11: unconnected-(U14-D2--Pad11) -> /HDMI_OUT/HDMI0_D1_P
- U14 pad 12: unconnected-(U14-D3+-Pad12) -> /HDMI_OUT/HDMI0_D2_N
- U14 pad 13: unconnected-(U14-D3--Pad13) -> /HDMI_OUT/HDMI0_D2_P
- U14 pad 14: unconnected-(U14-HPD-Pad14) -> /HDMI_OUT/HDMI0_HDP
- U14 pad 16: unconnected-(U14-SEL1-Pad16) -> /MCU/HDMI_SEL1
- U14 pad 17: unconnected-(U14-SEL2-Pad17) -> /MCU/HDMI_SEL2
- U14 pad 19: unconnected-(U14-HPD_A-Pad19) -> /HDMI_OUT/HDMI2_HPD
- U14 pad 2: unconnected-(U14-EN-Pad2) -> /MCU/HDMI_EN
- U14 pad 21: unconnected-(U14-HPD_B-Pad21) -> /HDMI_OUT/HDMI1_HPD
- U14 pad 22: unconnected-(U14-D3-B-Pad22) -> /HDMI_OUT/HDMI1_D2_P
- U14 pad 23: unconnected-(U14-D3+B-Pad23) -> /HDMI_OUT/HDMI1_D2_N
- U14 pad 24: unconnected-(U14-D2-B-Pad24) -> /HDMI_OUT/HDMI1_D1_P
- U14 pad 25: unconnected-(U14-D2+B-Pad25) -> /HDMI_OUT/HDMI1_D1_N
- U14 pad 26: unconnected-(U14-D1-B-Pad26) -> /HDMI_OUT/HDMI1_D0_P
- U14 pad 27: unconnected-(U14-D1+B-Pad27) -> /HDMI_OUT/HDMI1_D0_N
- U14 pad 28: unconnected-(U14-D0-B-Pad28) -> /HDMI_OUT/HDMI1_CLK_P
- U14 pad 29: unconnected-(U14-D0+B-Pad29) -> /HDMI_OUT/HDMI1_CLK_N
- U14 pad 3: unconnected-(U14-SCL-Pad3) -> /HDMI_OUT/HDMI0_SCL
- U14 pad 31: unconnected-(U14-D3-A-Pad31) -> /HDMI_OUT/HDMI2_D2_P
- U14 pad 32: unconnected-(U14-D3+A-Pad32) -> /HDMI_OUT/HDMI2_D2_N
- U14 pad 33: unconnected-(U14-D2-A-Pad33) -> /HDMI_OUT/HDMI2_D1_P
- U14 pad 34: unconnected-(U14-D2+A-Pad34) -> /HDMI_OUT/HDMI2_D1_N
- U14 pad 35: unconnected-(U14-D1-A-Pad35) -> /HDMI_OUT/HDMI2_D0_P
- U14 pad 36: unconnected-(U14-D1+A-Pad36) -> /HDMI_OUT/HDMI2_D0_N
- U14 pad 37: unconnected-(U14-D0-A-Pad37) -> /HDMI_OUT/HDMI2_CLK_P
- U14 pad 38: unconnected-(U14-D0+A-Pad38) -> /HDMI_OUT/HDMI2_CLK_N
- U14 pad 39: unconnected-(U14-SDA_B-Pad39) -> /HDMI_OUT/HDMI1_SDA
- U14 pad 4: unconnected-(U14-SDA-Pad4) -> /HDMI_OUT/HDMI0_SDA
- U14 pad 40: unconnected-(U14-SCL_B-Pad40) -> /HDMI_OUT/HDMI1_SCL
- U14 pad 41: unconnected-(U14-SDA_A-Pad41) -> /HDMI_OUT/HDMI2_SDA
- U14 pad 42: unconnected-(U14-SCL_A-Pad42) -> /HDMI_OUT/HDMI2_SCL
- U14 pad 5: unconnected-(U14-D0+-Pad5) -> /HDMI_OUT/HDMI0_CLK_N
- U14 pad 6: unconnected-(U14-D0--Pad6) -> /HDMI_OUT/HDMI0_CLK_P
- U14 pad 7: unconnected-(U14-D1+-Pad7) -> /HDMI_OUT/HDMI0_D0_N
- U14 pad 8: unconnected-(U14-D1--Pad8) -> /HDMI_OUT/HDMI0_D0_P
- U15 pad 1: Net-(U15-EN) -> Net-(U15-FB2)
- U15 pad 2: GND -> +5V
- U15 pad 3: Net-(U15-LX) -> Net-(U15-SW2)
- U15 pad 5: Net-(U15-FB/Vout) -> GND
- U16 pad 1: Net-(U16-EN) -> GND
- U16 pad 2: GND -> +3.3V
- U16 pad 3: Net-(U16-LX) -> +5V
- U16 pad 4: +5V -> +3.3V
- U6 pad 32: /TypeC2HDMI/HDMI_VBS -> +5V
- U6 pad 33: /TypeC2HDMI/HDMI_VBS -> +5V
- U6 pad 58: /TypeC2HDMI/GPIO_1 -> /MCU/GPIO_1
- U6 pad 59: /TypeC2HDMI/GPIO_2 -> /MCU/GPIO_2
- USB1 pad A4: /TypeC3.0Handle/HDMI_VBUS -> /Power/HDMI_VBUS
- USB1 pad A9: /TypeC3.0Handle/HDMI_VBUS -> /Power/HDMI_VBUS
- USB1 pad B4: /TypeC3.0Handle/HDMI_VBUS -> /Power/HDMI_VBUS
- USB1 pad B9: /TypeC3.0Handle/HDMI_VBUS -> /Power/HDMI_VBUS
- USB2 pad A4: /TypeC3.0Handle/TypeC_1_5V -> /Power/TypeC_1_5V
- USB2 pad A9: /TypeC3.0Handle/TypeC_1_5V -> /Power/TypeC_1_5V
- USB2 pad B4: /TypeC3.0Handle/TypeC_1_5V -> /Power/TypeC_1_5V
- USB2 pad B9: /TypeC3.0Handle/TypeC_1_5V -> /Power/TypeC_1_5V
- USB3 pad A4: /TypeC3.0Handle/TypeC_2_5V -> /Power/TypeC_2_5V
- USB3 pad A9: /TypeC3.0Handle/TypeC_2_5V -> /Power/TypeC_2_5V
- USB3 pad B4: /TypeC3.0Handle/TypeC_2_5V -> /Power/TypeC_2_5V
- USB3 pad B9: /TypeC3.0Handle/TypeC_2_5V -> /Power/TypeC_2_5V
- USB4 pad A4: /TypeC3.0Handle/TypeC_3_5V -> /Power/TypeC_3_5V
- USB4 pad A9: /TypeC3.0Handle/TypeC_3_5V -> /Power/TypeC_3_5V
- USB4 pad B4: /TypeC3.0Handle/TypeC_3_5V -> /Power/TypeC_3_5V
- USB4 pad B9: /TypeC3.0Handle/TypeC_3_5V -> /Power/TypeC_3_5V
- USB5 pad A4: /TypeC3.0Handle/TypeC_4_5V -> /Power/TypeC_4_5V
- USB5 pad A9: /TypeC3.0Handle/TypeC_4_5V -> /Power/TypeC_4_5V
- USB5 pad B4: /TypeC3.0Handle/TypeC_4_5V -> /Power/TypeC_4_5V
- USB5 pad B9: /TypeC3.0Handle/TypeC_4_5V -> /Power/TypeC_4_5V
- USB6 pad 18: /TypeC2HDMI/TMDS_5V -> /Power/TMDS_5V
- USB7 pad 1: unconnected-(USB7-TMDS_Data_2+-Pad1) -> /HDMI_OUT/HDMI0_D2_P
- USB7 pad 10: unconnected-(USB7-TMDS_Clock+-Pad10) -> /HDMI_OUT/HDMI0_CLK_P
- USB7 pad 11: unconnected-(USB7-TMDS_Clock_Shield-Pad11) -> GND
- USB7 pad 12: unconnected-(USB7-TMDS_Clock--Pad12) -> /HDMI_OUT/HDMI0_CLK_N
- USB7 pad 14: unconnected-(USB7-Reserved_(N.C.)-Pad14) -> GND
- USB7 pad 15: unconnected-(USB7-SCL-Pad15) -> /HDMI_OUT/HDMI0_SCL
- USB7 pad 16: unconnected-(USB7-SDA-Pad16) -> /HDMI_OUT/HDMI0_SDA
- USB7 pad 17: unconnected-(USB7-DDC/CEC_Ground-Pad17) -> GND
- USB7 pad 18: unconnected-(USB7-+5V_Power-Pad18) -> +5V
- USB7 pad 19: unconnected-(USB7-Hot_Plug_Detect-Pad19) -> /HDMI_OUT/HDMI0_HDP
- USB7 pad 2: unconnected-(USB7-TMDS_Data_2_Shield-Pad2) -> GND
- USB7 pad 20: unconnected-(USB7-GND-Pad20) -> GND
- USB7 pad 21: unconnected-(USB7-GND-Pad21) -> GND
- USB7 pad 22: unconnected-(USB7-GND-Pad22) -> GND
- USB7 pad 23: unconnected-(USB7-GND-Pad23) -> GND
- USB7 pad 3: unconnected-(USB7-TMDS_Data_2--Pad3) -> /HDMI_OUT/HDMI0_D2_N
- USB7 pad 4: unconnected-(USB7-TMDS_Data_1+-Pad4) -> /HDMI_OUT/HDMI0_D1_P
- USB7 pad 5: unconnected-(USB7-TMDS_Data_1_Shield-Pad5) -> GND
- USB7 pad 6: unconnected-(USB7-TMDS_Data_1--Pad6) -> /HDMI_OUT/HDMI0_D1_N
- USB7 pad 7: unconnected-(USB7-TMDS_Data_0+-Pad7) -> /HDMI_OUT/HDMI0_D0_P
- USB7 pad 8: unconnected-(USB7-TMDS_Data_0_Shield-Pad8) -> GND
- USB7 pad 9: unconnected-(USB7-TMDS_Data_0--Pad9) -> /HDMI_OUT/HDMI0_D0_N

Commit message: 开始PCB布局
Parts:
- moved C1 260.2 mm to (451.3, -1.75)
- moved C104 260.2 mm to (386.4, -37.0)
- moved C105 260.2 mm to (386.4, -34.3)
- moved C106 260.2 mm to (386.4, -31.6)
- moved C107 260.2 mm to (386.4, -28.9)
- moved C108 260.2 mm to (386.4, -26.3)
- moved C109 260.2 mm to (383.8, -0.50)
- moved C110 260.2 mm to (386.4, -23.6)
- moved C111 260.2 mm to (390.4, -37.0)
- moved C112 260.2 mm to (390.4, -34.3)
- moved C113 260.2 mm to (390.4, -31.6)
- moved C114 260.2 mm to (390.4, -28.9)
- moved C115 260.2 mm to (390.4, -26.3)
- moved C19 260.2 mm to (463.4, -1.75)
- moved C2 260.2 mm to (451.3, 0.93)
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Other:
- board size 8.2 x 0.8 mm -> 100 x 50 mm
